File: Anti-Spark Switch.kicad_sch (KiCad schematic)
At the start: 16 parts, among them J1 Conn_01x01, J2 Conn_01x01, J4 Conn_01x01, J6 Conn_01x01, J7 Conn_01x02, Q1 IRF3205, Q2 IRF3205, Q3 IRF3205, SW1 SW_Push

Commit message: pcb laid out
Parts:
- removed SW1: SW_Push, symbol Switch:SW_Push
- added J3: Conn_01x02, Connector_JST:JST_PH_S2B-PH-K_1x02_P2.00mm_Horizontal, symbol Connector_Generic:Conn_01x02
- added J5: XT60PW-F, Connector_AMASS:AMASS_XT60PW-F_1x02_P7.20mm_Horizontal, symbol XT60PW-F:XT60PW-F
- added J8: XT60PW-M, Connector_AMASS:AMASS_XT60PW-M_1x02_P7.20mm_Horizontal, symbol XT60PW-F:XT60PW-F
- C1: footprint (none) -> Capacitor_SMD:C_0805_2012Metric_Pad1.18x1.45mm_HandSolder
- D1: footprint (none) -> Diode_SMD:D_SMA-SMB_Universal_Handsoldering
- J1, J2, J4, J6: footprint (none) -> Pad:1PAD_12x7mm
- J7: footprint (none) -> Connector_JST:JST_PH_S2B-PH-K_1x02_P2.00mm_Horizontal
- Q1, Q2, Q3: value IRF3205 -> DMT10H010LK3; footprint Package_TO_SOT_THT:TO-220-3_Vertical -> Package_TO_SOT_SMD:TO-252-2; symbol Transistor_FET:IRF3205 -> Transistor_FET:DMN10H700S
- R1, R2, R3: footprint (none) -> Resistor_SMD:R_0805_2012Metric_Pad1.20x1.40mm_HandSolder
- R4, R5: footprint (none) -> Resistor_SMD:R_2512_6332Metric_Pad1.40x3.35mm_HandSolder
Connections:
- net GND: now also J3.1 (Pin_1), J8.1
- net VCC: now also J5.2, J8.2
- net at C1.2, D1.1 (K), Q1.1 (G)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: now also J3.2 (Pin_2)
- net at J1.1 (Pin_1), J7.2 (Pin_2), Q1.2 (D)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: now also J5.1
Other:
- moved on the sheet: J4, J6
